File: PCB/BlinkyBoard.kicad_pcb (KiCad board)
At the start: 2 copper layers, 104.9 x 95 mm, 21 parts, among them J1 Conn_01x02_Socket, J2 Conn_01x01_Socket, U1 NE555P, U2 4017

Commit message: Add files via upload
Parts:
- moved D3 3.82 mm to (137.6, 114.1)
- moved D4 3.48 mm to (204.6, 114.1)
- moved D6 3.11 mm to (125.7, 54.2)
- moved D10 2.55 mm to (191.5, 69.6)
- moved D5 2.53 mm to (210.4, 88.8)
- moved J1 2.47 mm to (193.3, 101.6)
- moved D9 2.47 mm to (216.3, 53.7)
- moved J2 2.43 mm to (150.8, 100.3)
- moved D2 2.33 mm to (149.2, 68.4)
- moved D8 2.33 mm to (188.7, 127.2)
- moved D1 2.11 mm to (131.6, 89.8)
- moved D7 1.23 mm to (153.1, 127.4)
- moved G*** 0.95 mm to (198.0, 93.3)
- moved G*** 0.88 mm to (145.9, 92.8)
- moved R1 0.19 mm to (175.8, 99.9)
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Routing:
- net Net-(D6-A): track 60.2 -> 57.1 mm
- net Net-(D3-A): track 40.2 -> 37.3 mm
- net Net-(D5-A): track 38.6 -> 36.0 mm
- net Net-(D8-A): track 34.4 -> 36.7 mm
- net Net-(D10-A): track 30.4 -> 28.1 mm
- net Net-(D1-A): track 39.7 -> 37.4 mm
- net Net-(D1-K): track 9.50 -> 7.31 mm
- net Net-(D9-A): track 55.3 -> 53.2 mm
- net Net-(D4-A): track 38.3 -> 36.3 mm
- net Net-(D2-A): track 36.1 -> 34.2 mm
- net +5V: track 51.8 -> 50.2 mm
- net Net-(D7-A): track 36.7 -> 37.7 mm
Other:
- board size 104.9 x 95 mm -> 99.2 x 89.8 mm
